Commit message: changes 1.0

File: src/mini-ros2/robots/descriptions/mini_description/xacro/gazebo.xacro (robot description, xacro)
@@ -366,5 +366,43 @@
       xyz="0 0 0" />
   </joint>
+  <!-- GAZEBO LASER -->
+  <gazebo reference="lidar_link">
+    <material>Gazebo/FlatBlack</material>
+    <sensor type="ray" name="lds_lfcd_sensor">
+      <pose>0 0 0 0 0 0</pose>
+      <always_on>true</always_on>
+      <update_rate>10.0</update_rate>
+      <visualize>true</visualize>
+      <ray>
+        <scan>
+          <horizontal>
+            <samples>360</samples>
+            <resolution>1</resolution>
+            <min_angle>0.0</min_angle>
+            <max_angle>6.28319</max_angle>
+          </horizontal>
+        </scan>
+        <range>
+          <min>0.120</min>
+          <max>3.5</max>
+          <resolution>0.015</resolution>
+        </range>
+        <noise>
+          <type>gaussian</type>
+          <mean>0.0</mean>
+          <stddev>0.01</stddev>
+        </noise>
+      </ray>
+      <plugin name="gazebo_ros_lds_lfcd_controller" filename="libgazebo_ros_ray_sensor.so">
+        <ros>
+          <namespace></namespace>
+          <remapping>~/out:=scan</remapping>
+        </ros>
+        <output_type>sensor_msgs/LaserScan</output_type>
+      </plugin>
+    </sensor>
+  </gazebo>
   <!-- Lidar Plugin-->
+  <!--
   <gazebo reference="lidar_link">
   <sensor name="lidar" type="ray">
@@ -395,5 +433,5 @@
     <plugin name="scan" filename="libgazebo_ros_ray_sensor.so">
       <ros>
-        <remapping>~/out:=scan_4</remapping>
+        <remapping>~/out:=scan</remapping>
       </ros>
       <output_type>sensor_msgs/LaserScan</output_type>
@@ -401,4 +439,4 @@
     </plugin>
   </sensor>
-  </gazebo>
+  </gazebo> -->
 </robot>

File: src/mini-ros2/robots/descriptions/mini_description/xacro/robot.xacro (robot description, xacro)
@@ -60,5 +60,5 @@
     </joint> -->
     <joint name="imu_joint" type="fixed">
-        <parent link="trunk"/>
+        <parent link="base_link"/>
         <child link="imu_link"/>
         <origin rpy="0 0 0" xyz="0 0 0"/>
